Commit message: Add the nice STL so the visual is correct, add a sample Jackal config file, add frames for each of the camera lenses

File: urdf/omni_60.urdf.xacro (robot description, xacro)
@@ -2,23 +2,20 @@
 <robot xmlns:xacro="http://wiki.ros.org/xacro">
   <xacro:macro name="omni_60" params="parent name='omni_60' *origin">
-    <!--
-      TODO: replace this cylinder with a nice mesh that looks more accurate
-      TODO: add links for each camera frame so we can tag the frame_id for each of the 5 image streams
-    -->
     <link name="${name}_base_link">
       <visual>
         <geometry>
-          <cylinder radius="0.0525" length="0.07" />
+          <mesh filename="package://occam_ros/meshes/omni_60.stl" />
         </geometry>
-        <origin xyz="0 0 0.035" rpy="0 0 0" />
+        <origin xyz="0 0 0" rpy="${pi/2} 0 -${pi/2}" />
         <material name="navy">
-          <color rgba="0 0 0.5 1" />
+          <color rgba="0.1 0.1 0.7 1" />
         </material>
       </visual>
+      <!-- For simplicity, treat the collision model as a cylinder -->
       <collision>
         <geometry>
-          <cylinder radius="0.0525" length="0.07" />
+          <cylinder radius="0.05225" length="0.0535" />
         </geometry>
-        <origin xyz="0 0 ${0.0525/2}" rpy="0 0 0" />
+        <origin xyz="0 0 ${0.0535/2}" rpy="0 0 0" />
       </collision>
     </link>
@@ -28,4 +25,70 @@
       <xacro:insert_block name="origin" />
     </joint>
+    <!--
+      The 5 cameras are arrayed radially, so define 2 links per camera: one in the middle with the correct yaw
+      and a second for the actual image frame.  This lets us basically use polar coordinates, instead of
+      caluclating XYZ transforms for each frame
+    -->
+    <!-- TODO double-check which way around the lenses are enumerated on an actual camera -->
+    <link name="${name}_camera1_link"/>
+    <link name="${name}_camera2_link"/>
+    <link name="${name}_camera3_link"/>
+    <link name="${name}_camera4_link"/>
+    <link name="${name}_camera5_link"/>
+    <link name="${name}_camera1_internal_link"/>
+    <link name="${name}_camera2_internal_link"/>
+    <link name="${name}_camera3_internal_link"/>
+    <link name="${name}_camera4_internal_link"/>
+    <link name="${name}_camera5_internal_link"/>
+    <joint name="${name}_camera3_orientation_joint" type="fixed">
+      <parent link="${name}_base_link" />
+      <child link="${name}_camera3_internal_link" />
+      <origin xyz="0 0 0.026" rpy="0 0 0" />
+    </joint>
+    <joint name="${name}_camera2_orientation_joint" type="fixed">
+      <parent link="${name}_camera3_internal_link" />
+      <child link="${name}_camera2_internal_link" />
+      <origin xyz="0 0 0" rpy="0 0 ${2*pi/5}" />
+    </joint>
+    <joint name="${name}_camera1_orientation_joint" type="fixed">
+      <parent link="${name}_camera3_internal_link" />
+      <child link="${name}_camera1_internal_link" />
+      <origin xyz="0 0 0" rpy="0 0 ${4*pi/5}" />
+    </joint>
+    <joint name="${name}_camera4_orientation_joint" type="fixed">
+      <parent link="${name}_camera3_internal_link" />
+      <child link="${name}_camera4_internal_link" />
+      <origin xyz="0 0 0" rpy="0 0 -${2*pi/5}" />
+    </joint>
+    <joint name="${name}_camera5_orientation_joint" type="fixed">
+      <parent link="${name}_camera3_internal_link" />
+      <child link="${name}_camera5_internal_link" />
+      <origin xyz="0 0 0" rpy="0 0 -${4*pi/5}" />
+    </joint>
+    <joint name="${name}_camera3_joint" type="fixed">
+      <parent link="${name}_camera3_internal_link" />
+      <child link="${name}_camera3_link" />
+      <origin xyz="0.05225 0 0" rpy="0 0 0" />
+    </joint>
+    <joint name="${name}_camera2_joint" type="fixed">
+      <parent link="${name}_camera2_internal_link" />
+      <child link="${name}_camera2_link" />
+      <origin xyz="0.05225 0 0" rpy="0 0 0" />
+    </joint>
+    <joint name="${name}_camera1_joint" type="fixed">
+      <parent link="${name}_camera1_internal_link" />
+      <child link="${name}_camera1_link" />
+      <origin xyz="0.05225 0 0" rpy="0 0 0" />
+    </joint>
+    <joint name="${name}_camera4_joint" type="fixed">
+      <parent link="${name}_camera4_internal_link" />
+      <child link="${name}_camera4_link" />
+      <origin xyz="0.05225 0 0" rpy="0 0 0" />
+    </joint>
+    <joint name="${name}_camera5_joint" type="fixed">
+      <parent link="${name}_camera5_internal_link" />
+      <child link="${name}_camera5_link" />
+      <origin xyz="0.05225 0 0" rpy="0 0 0" />
+    </joint>
   </xacro:macro>
 </robot>
